File: modularPCB/Modular/Casillero.sch (EAGLE design)
At the start: 41 parts

Commit message: Actualización de pcbs
Parts:
- removed ALARMA, DISPONIBLE, EMISOR, EMISOR1, LED1, LED2, LED3, LED4, OCUPADO, RECEPTOR, RECEPTOR1: (no value), led:LED3MM
- removed CHAPA-DATA, CHAPA-VOL: (no value), pinhead:PINHD-1X2
- removed D1: 1N4004, diode:1N4004
- removed R-ALARMA, R-DISPONIBLE, R-GAL, R-INFRA-LED, R-INFRA-LED1, R-OCUPADO, R-UL: 220, rcl:R-EU_0204/7
- removed R-CHAPA, R-G1, R-G2: 1k, rcl:R-EU_0204/7
- removed R-CHAPA2: 330, rcl:R-EU_0204/7
- removed R-EMISOR, R-EMISOR1: 380, rcl:R-EU_0204/7
- removed R-INFRA, R-INFRA1, R-RECEPTOR, R-RECEPTOR1: 22K, rcl:R-EU_0204/7
- removed U$2: ULTRASONICO, MODULAR:ULTRASONICO
- removed U$4, U$6, U$7: 2N2222, MODULAR:2N2222
- removed U$5: RELEY, MODULAR:RELEY
- added JP2, JP3: (no value), pinhead:PINHD-1X1
- added R-B, R-G, R-R: 220, rcl:R-EU_0204/7
- added SG1: F/CM12P, buzzer:F/CM12P
- added SV1, SV2: (no value), con-lstb:MA04-2
- added X1, X7: 22-23-2041, con-molex:22-23-2041
- added X2, X3: 22-23-2031, con-molex:22-23-2031
- added X4, X5, X6: 22-23-2021, con-molex:22-23-2021
- JP1: device pinhead:PINHD-1X3 -> pinhead:PINHD-1X1
- U$3: value HX-711 -> LEDRGB; device MODULAR:HX-711 -> MODULAR:LEDRGB
Connections:
- removed net DATO-CHAPA: CHAPA-DATA.1, R-CHAPA2.2, U$1.D27
- removed net DT-GALGA: U$1.D18, U$3.DT
- removed net ECHO-ULTRASONICO: U$1.D22, U$2.ECHO
- removed net GND1: U$1.GND@1
- removed net LIBRE: U$1.D15
- removed net LIBRE1: U$1.D5
- removed net LIBRE2: U$1.D25
- removed net N$1: LED1.C, R-UL.2
- removed net N$10: D1.A, U$4.C, U$5.B1
- removed net N$13: JP1.1, U$3.A+
- removed net N$14: JP1.2, R-G1.2, U$3.E-
- removed net N$15: JP1.3, R-G2.2, U$3.E+
- removed net N$16: R-G1.1, R-G2.1, U$3.A-
- removed net N$20: EMISOR.A, R-EMISOR.1
- removed net N$24: CHAPA-VOL.1, U$5.NA
- removed net N$30: R-RECEPTOR.1, RECEPTOR.C, U$6.B
- removed net N$31: LED3.A, R-INFRA-LED.1
- removed net N$32: DISPONIBLE.C, R-DISPONIBLE.2
- removed net N$33: ALARMA.C, R-ALARMA.2
- removed net N$34: R-SENSADO.2, SENSADO.C
- removed net N$8: LED2.C, R-GAL.2
- removed net N$9: R-CHAPA.1, U$4.B
- removed net PULSO-ALARMA: ALARMA.A, U$1.D14
- removed net PULSO-CHAPA: R-CHAPA.2, U$1.D26
- removed net PULSO-DISPONIBLE: DISPONIBLE.A, U$1.D12
- removed net PULSO-GALGA: LED2.A, U$1.D21
- removed net PULSO-INFRA: R-INFRA-LED.2, R-INFRA-LED1.2, R-INFRA.1, R-INFRA1.1, U$1.D2, U$6.E, U$7.E
- removed net PULSO-OCUPADO: OCUPADO.A, U$1.D13
- removed net PULSO-SENSADO: SENSADO.A, U$1.D4
- removed net PULSO-ULTRASONICO: LED1.A, U$1.D32
- removed net PURA-ENTRADA: U$1.D34
- removed net SCK-GALGA: U$1.D19, U$3.SCK
- removed net TRIG-ULTRASONICO: U$1.D23, U$2.TRIG
- removed net VF: D1.C, U$5.B2, U$5.IN
- new net BUZZER: SG1.1, U$1.D27
- new net CERRADURA_CTRL: U$1.D25, X6-2.S
- new net CERRADURA_VCC: U$1.D26, X6-1.S
- new net GA_DT: U$1.D19, X3-2.S
- new net GA_LED: U$1.D21, X3-1.S
- new net GA_SCK: U$1.D18, X3-3.S
- new net IR: JP1.1, U$1.D34
- new net LCD_SCL: U$1.D5, X5-2.S
- new net LCD_SDA: U$1.D15, X5-1.S
- new net LED_B: R-B.2, U$1.D14, X1-4.S, X7-2.S
- new net LED_G: R-G.2, U$1.D12, X1-3.S, X7-3.S
- new net LED_R: R-R.2, U$1.D13, X1-2.S, X7-4.S
- new net SENSADO_LED: JP2.1, R-SENSADO.2, U$1.D4, X4-2.S
- new net UL_ECHO: U$1.D22, X2-2.S
- new net UL_LED: U$1.D32, X2-1.S
- new net UL_TRG: U$1.D23, X2-3.S
- new net WIFI_LED: U$1.D2
- net 3V3: now also SV1.1, SV1.3, SV1.5, SV1.7; no longer CHAPA-DATA.2, R-EMISOR.2, R-EMISOR1.2, R-RECEPTOR.2, R-RECEPTOR1.2, U$3.VCC
- net GND: now also SENSADO.C, SG1.2, SV1.2, SV1.4, SV1.6, SV1.8, SV2.2, SV2.4, SV2.6, SV2.8, U$1.GND@1, U$3.CATODO, X1-1.S, X4-1.S, X7-1.S; no longer CHAPA-VOL.2, EMISOR.C, EMISOR1.C, LED3.C, LED4.C, R-ALARMA.1, R-CHAPA2.1, R-DISPONIBLE.1, R-GAL.1, R-INFRA.2, R-INFRA1.2, R-OCUPADO.1, R-SENSADO.1, R-UL.1, RECEPTOR.A, RECEPTOR1.A, U$2.GND, U$3.GND, U$4.E
- net N$2: now also R-R.1, U$3.R; no longer EMISOR1.A, R-EMISOR1.1
- net N$3: now also R-G.1, U$3.G; no longer OCUPADO.C, R-OCUPADO.2
- net N$4: now also R-B.1, U$3.B; no longer R-RECEPTOR1.1, RECEPTOR1.C, U$7.B
- net N$7: now also R-SENSADO.1, SENSADO.A; no longer LED4.A, R-INFRA-LED1.1
- net VIN: now also SV2.1, SV2.3, SV2.5, SV2.7; no longer U$2.VCC, U$6.C, U$7.C
Other:
- note removed: "CELDA DE CARGA"
- note removed: "CIRCUITO CHAPA"
- note removed: "INFRARROJO"
- note removed: "MODULO ULTRASONICO"
- moved on the sheet: R-SENSADO, SENSADO
