File: modularPCB/Modular/PCB-MODULOS/SENSORES/Infrarrojo.sch (EAGLE design)
At the start: 9 parts

Commit message: Corrección de errores en pcbs
Parts:
- renumbered U$6 to U$1
Changed lines of the file:
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@@
 <parts>
 <part name="R1" library="rcl" library_urn="urn:adsk.eagle:library:334" deviceset="R-EU_" device="0204/7" package3d_urn="urn:adsk.eagle:package:23498/2" value="380"/>
-<part name="U$6" library="MODULAR" deviceset="2N2222" device=""/>
 <part name="D1E" library="led" library_urn="urn:adsk.eagle:library:259" deviceset="LED" device="3MM" package3d_urn="urn:adsk.eagle:package:15797/1"/>
 <part name="R2" library="rcl" library_urn="urn:adsk.eagle:library:334" deviceset="R-EU_" device="0204/7" package3d_urn="urn:adsk.eagle:package:23498/2" value="22K"/>
@@
 <part name="R4" library="rcl" library_urn="urn:adsk.eagle:library:334" deviceset="R-EU_" device="0204/7" package3d_urn="urn:adsk.eagle:package:23498/2" value="220"/>
 <part name="JP1" library="pinhead" library_urn="urn:adsk.eagle:library:325" deviceset="PINHD-1X4" device="" package3d_urn="urn:adsk.eagle:package:22407/2"/>
+<part name="U$1" library="MODULAR" deviceset="2N2222" device=""/>
 </parts>
 <sheets>
@@
 <attribute name="VALUE" x="10.922" y="46.99" size="1.778" layer="96" rot="R90"/>
 </instance>
-<instance part="U$6" gate="G$1" x="40.64" y="48.26" smashed="yes"/>
 <instance part="D1E" gate="G$1" x="7.62" y="40.64" smashed="yes">
 <attribute name="NAME" x="1.524" y="40.132" size="1.778" layer="95" rot="R270"/>
@@
 <attribute name="VALUE" x="57.15" y="67.31" size="1.778" layer="96" rot="R90"/>
 </instance>
+<instance part="U$1" gate="G$1" x="40.64" y="48.26" smashed="yes"/>
 </instances>
 <busses>
@@
 <net name="VIN" class="0">
 <segment>
-<pinref part="U$6" gate="G$1" pin="C"/>
 <wire x1="43.18" y1="53.34" x2="43.18" y2="55.88" width="0.1524" layer="91"/>
 <junction x="43.18" y="55.88"/>
@@
 <pinref part="JP1" gate="A" pin="3"/>
 <wire x1="49.53" y1="57.15" x2="49.53" y2="71.12" width="0.1524" layer="91"/>
+<pinref part="U$1" gate="G$1" pin="C"/>
 </segment>
 </net>
@@
 <pinref part="D2R" gate="G$1" pin="C"/>
 <wire x1="25.4" y1="45.72" x2="25.4" y2="43.18" width="0.1524" layer="91"/>
-<pinref part="U$6" gate="G$1" pin="B"/>
+<pinref part="U$1" gate="G$1" pin="B"/>
 <wire x1="25.4" y1="43.18" x2="25.4" y2="40.64" width="0.1524" layer="91"/>
 <wire x1="33.02" y1="43.18" x2="25.4" y2="43.18" width="0.1524" layer="91"/>
@@
 <segment>
 <pinref part="R3" gate="G$1" pin="1"/>
-<pinref part="U$6" gate="G$1" pin="E"/>
 <wire x1="43.18" y1="25.4" x2="43.18" y2="27.94" width="0.1524" layer="91"/>
 <wire x1="43.18" y1="27.94" x2="43.18" y2="30.48" width="0.1524" layer="91"/>
@@
 <pinref part="JP1" gate="A" pin="4"/>
 <wire x1="52.07" y1="57.15" x2="52.07" y2="71.12" width="0.1524" layer="91"/>
+<pinref part="U$1" gate="G$1" pin="E"/>
 </segment>
 </net>
